File: schemat.brd (EAGLE design)
At the start: 160 x 100 mm, 35 parts, among them IC1 STM32F10XCXT6, X1 RASPI_BOARD_B+#_E4P

Commit message: SAE_ADV_PCB_V2
Parts:
- moved JP2 49.0 mm to (48.9, 50.8)
- moved C9 44.7 mm to (54.6, 35.6)
- moved C5 41.1 mm to (51.2, 26.7), turned to 270 degrees
- moved C8 34.8 mm to (44.5, 47.6), flipped to the bottom, turned to 180 degrees
- moved C7 33.0 mm to (43.2, 38.7), turned to 225 degrees
- moved C6 30.5 mm to (40.6, 36.2), turned to 225 degrees
- moved C10 30.0 mm to (41.1, 50.4), turned to 225 degrees
- moved C15 27.4 mm to (59.4, 11.9), flipped to the bottom, turned to 90 degrees
- moved JP4 26.1 mm to (59.1, 37.5)
- moved JP13 20.3 mm to (46.2, 11.0), turned to 180 degrees
- moved C17 20.1 mm to (65.8, 15.7)
- moved C16 17.8 mm to (56.9, 9.40)
- moved C14 17.4 mm to (67.8, 19.9), flipped to the bottom
- moved JP9 16.5 mm to (66.7, 40.6)
- moved JP5 15.1 mm to (66.7, 25.4)
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Connections:
- net PWM_INPUT_1: now also JP12.2; no longer JP12.1
- net PWM_INPUT_2: now also JP12.1; no longer JP12.2
- net PWM_INPUT_4: now also IC1.10; no longer IC1.38
- net RPI_SIGNAL_1: now also IC1.41; no longer IC1.42
- net RPI_SIGNAL_2: now also IC1.39; no longer IC1.41
- net RPI_SIGNAL_3: now also IC1.42; no longer IC1.40
- net RPI_SIGNAL_4: now also IC1.40; no longer IC1.39
Routing:
- net BOOT_0: track 72.7 -> 15.7 mm, vias 2 -> 1
- net +3V3: track 117.6 -> 62.6 mm, vias 2 -> 1
- net PWM_OUTPUT_1: track 34.1 -> 15.4 mm, vias 2 -> 1
- net PWM_OUTPUT_0: track 37.1 -> 22.6 mm, vias 4 -> 1
- net PWM_INPUT_4: track 29.4 -> 15.0 mm, vias 0 -> 1
- net SWCLK: track 23.0 -> 8.97 mm, vias 2 -> 0
- net RPI_SIGNAL_2: track 9.16 -> 22.7 mm
- net RPI_SIGNAL_1: track 8.95 -> 22.1 mm
- net SWDIO: track 19.6 -> 7.26 mm, vias 2 -> 0
- net +5V_SERWO: track 60.6 -> 48.8 mm
- net RPI_SIGNAL_3: track 14.4 -> 24.8 mm
- net RPI_SIGNAL_4: track 15.8 -> 25.5 mm
- net +5V: track 47.3 -> 37.9 mm, vias 1 -> 0
- net NRST: track 22.0 -> 12.7 mm
- net PWM_INPUT_3: track 16.1 -> 9.86 mm
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