File: schemat.sch (EAGLE design)
At the start: 20 parts, among them IC1 STM32F10XCXT6, X1 RASPI_BOARD_B+#_E4P

Commit message: SKOŃCZONY SCHEMAT
Parts:
- added C14, C15: 100nF, rcl:C-EUC0603
- added C16, C17: 330uF, rcl:CPOL-EUE3.5-10
- added JP10, JP11, JP3, JP4, JP5, JP6, JP7, JP8, JP9: (no value), pinhead:PINHD-1X3
- added JP12: (no value), pinhead:PINHD-1X5
- added JP13: (no value), pinhead:PINHD-1X2
Connections:
- new net +5V_SERWO: C14.1, C15.1, C16.+, C17.+, JP10.2, JP13.1, JP5.2, JP6.2, JP8.2, JP9.2
- new net +5_SERWO: JP7.2
- new net PWM_INPUT_1: IC1PORTB_L.PB0, JP12.1
- new net PWM_INPUT_2: IC1PORTA_L.PA6, JP12.2
- new net PWM_INPUT_3: IC1PORTB_H.PB10, JP12.3
- new net PWM_INPUT_4: IC1PORTA_H.PA15, JP12.4
- new net PWM_OUTPUT_0: JP9.1, X1.GPIO12
- new net PWM_OUTPUT_1: JP10.1, X1.GPIO13
- new net RPI_SIGNAL_1: IC1PORTB_L.PB6, X1.GPIO19
- new net RPI_SIGNAL_2: IC1PORTB_L.PB5, X1.GPIO26
- new net RPI_SIGNAL_3: IC1PORTB_L.PB4, X1.GPIO16
- new net RPI_SIGNAL_4: IC1PORTB_L.PB3, X1.GPIO20
- new net SERWO_PWM_OUTPUT4: JP5.1
- new net SERWO_PWM_OUTPUT_1: IC1PORTA_H.PA11, JP8.1
- new net SERWO_PWM_OUTPUT_2: IC1PORTA_H.PA10, JP7.1
- new net SERWO_PWM_OUTPUT_3: IC1PORTA_H.PA9, JP6.1
- new net SERWO_PWM_OUTPUT_4: IC1PORTA_H.PA8
- new net STM32_SIGNAL_1: IC1PORTB_H.PB9, X1.GPIO17, X1.GPIO22
- new net STM32_SIGNAL_2: IC1PORTB_H.PB8, X1.GPIO27
- new net STM32_SIGNAL_3: IC1PORTB_L.PB7
- new net SWCLK: IC1PORTA_H.PA14, JP4.2
- new net SWDIO: JP4.1
- new net SWIDO: IC1PORTA_H.PA13
- new net UART_RX: IC1PORTA_L.PA3, JP11.2, JP3.2
- new net UART_RXD: X1.RXD
- new net UART_TX: IC1PORTA_L.PA2, JP11.1, JP3.1
- new net UART_TXD: X1.TXD
- net GND: now also C14.2, C15.2, C16.-, C17.-, JP10.3, JP11.3, JP12.5, JP13.2, JP3.3, JP4.3, JP5.3, JP6.3, JP7.3, JP8.3, JP9.3
Other:
- note added: "Fitracja zasilania serwo"
- note added: "HEADER_1"
- note added: "HEADER_10"
- note added: "HEADER_11"
- note added: "HEADER_2"
- note added: "HEADER_3"
- note added: "HEADER_4"
- note added: "HEADER_5"
- note added: "HEADER_6"
- note added: "HEADER_7"
- note added: "HEADER_8"
- note added: "HEADER_9"
- note added: "Header X"
- note added: "Przełaczanie trybu pracy"
- note added: "Układ rezonatora 8 MHz"
- note added: "Zabezpieczenie obwodu NRST (reset)"
- note removed: "Filtracja/obwód załączenia NRST"
- moved on the sheet: C11, JP1, JP2, S1

Commit message: PCB V1
Connections:
- removed net +5_SERWO: JP7.2
- removed net N$3: C11.2, S1.2
- removed net SERWO_PWM_OUTPUT4: JP5.1
- removed net SWIDO: IC1PORTA_H.PA13
- net +5V_SERWO: now also JP7.2
- net GND: now also C11.2, S1.2
- net SERWO_PWM_OUTPUT_4: now also JP5.1
- net STM32_SIGNAL_1: no longer X1.GPIO22
- net STM32_SIGNAL_3: now also X1.GPIO22
- net SWDIO: now also IC1PORTA_H.PA13
- net UART_RX: no longer JP11.2
- net UART_RXD: now also JP11.2
- net UART_TX: no longer JP11.1
- net UART_TXD: now also JP11.1

Commit message: SAE_ADV_PCB_V2
Connections:
- net PWM_INPUT_1: now also JP12.2; no longer JP12.1
- net PWM_INPUT_2: now also JP12.1; no longer JP12.2
- net PWM_INPUT_4: now also IC1PORTA_L.PA0; no longer IC1PORTA_H.PA15
- net RPI_SIGNAL_1: now also IC1PORTB_L.PB5; no longer IC1PORTB_L.PB6
- net RPI_SIGNAL_2: now also IC1PORTB_L.PB3; no longer IC1PORTB_L.PB5
- net RPI_SIGNAL_3: now also IC1PORTB_L.PB6; no longer IC1PORTB_L.PB4
- net RPI_SIGNAL_4: now also IC1PORTB_L.PB4; no longer IC1PORTB_L.PB3
Changed lines of the file:
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@@
 <?xml version="1.0" encoding="utf-8"?>
 <!DOCTYPE eagle SYSTEM "eagle.dtd">
-<eagle version="9.4.2">
+<eagle version="9.5.2">
 <drawing>
 <settings>
@@
 <net name="PWM_INPUT_1" class="0">
 <segment>
+<pinref part="IC1" gate="PORTB_L" pin="PB0"/>
+<wire x1="22.86" y1="91.44" x2="27.94" y2="91.44" width="0.1524" layer="91"/>
+<label x="25.4" y="91.44" size="1.778" layer="95"/>
+</segment>
+<segment>
+<pinref part="JP12" gate="A" pin="2"/>
+<wire x1="101.6" y1="152.4" x2="83.82" y2="152.4" width="0.1524" layer="91"/>
+<label x="78.74" y="152.4" size="1.778" layer="95"/>
+</segment>
+</net>
+<net name="PWM_INPUT_2" class="0">
+<segment>
+<pinref part="IC1" gate="PORTA_L" pin="PA6"/>
+<wire x1="-12.7" y1="76.2" x2="-17.78" y2="76.2" width="0.1524" layer="91"/>
+<label x="-30.48" y="76.2" size="1.778" layer="95"/>
+</segment>
+<segment>
 <pinref part="JP12" gate="A" pin="1"/>
 <wire x1="101.6" y1="154.94" x2="83.82" y2="154.94" width="0.1524" layer="91"/>
 <label x="78.74" y="154.94" size="1.778" layer="95"/>
 </segment>
-<segment>
-<pinref part="IC1" gate="PORTB_L" pin="PB0"/>
-<wire x1="22.86" y1="91.44" x2="27.94" y2="91.44" width="0.1524" layer="91"/>
-<label x="25.4" y="91.44" size="1.778" layer="95"/>
-</segment>
-</net>
-<net name="PWM_INPUT_2" class="0">
-<segment>
-<pinref part="JP12" gate="A" pin="2"/>
-<wire x1="101.6" y1="152.4" x2="83.82" y2="152.4" width="0.1524" layer="91"/>
-<label x="78.74" y="152.4" size="1.778" layer="95"/>
-</segment>
-<segment>
-<pinref part="IC1" gate="PORTA_L" pin="PA6"/>
-<wire x1="-12.7" y1="76.2" x2="-17.78" y2="76.2" width="0.1524" layer="91"/>
-<label x="-30.48" y="76.2" size="1.778" layer="95"/>
-</segment>
 </net>
 <net name="PWM_INPUT_3" class="0">
@@
 </segment>
 <segment>
-<pinref part="IC1" gate="PORTA_H" pin="PA15"/>
-<wire x1="-12.7" y1="48.26" x2="-17.78" y2="48.26" width="0.1524" layer="91"/>
-<label x="-33.02" y="48.26" size="1.778" layer="95"/>
+<pinref part="IC1" gate="PORTA_L" pin="PA0"/>
+<wire x1="-12.7" y1="91.44" x2="-17.78" y2="91.44" width="0.1524" layer="91"/>
+<label x="-30.48" y="91.44" size="1.778" layer="95"/>
 </segment>
 </net>
@@
 <net name="RPI_SIGNAL_4" class="0">
 <segment>
+<pinref part="X1" gate="G$1" pin="GPIO20"/>
+<wire x1="91.44" y1="17.78" x2="86.36" y2="17.78" width="0.1524" layer="91"/>
+<label x="68.58" y="17.78" size="1.778" layer="95"/>
+</segment>
+<segment>
+<pinref part="IC1" gate="PORTB_L" pin="PB4"/>
+<wire x1="22.86" y1="81.28" x2="27.94" y2="81.28" width="0.1524" layer="91"/>
+<label x="25.4" y="81.28" size="1.778" layer="95"/>
+</segment>
+</net>
+<net name="RPI_SIGNAL_3" class="0">
+<segment>
+<pinref part="X1" gate="G$1" pin="GPIO16"/>
+<wire x1="91.44" y1="22.86" x2="86.36" y2="22.86" width="0.1524" layer="91"/>
+<label x="68.58" y="22.86" size="1.778" layer="95"/>
+</segment>
+<segment>
+<pinref part="IC1" gate="PORTB_L" pin="PB6"/>
+<wire x1="22.86" y1="76.2" x2="27.94" y2="76.2" width="0.1524" layer="91"/>
+<label x="25.4" y="76.2" size="1.778" layer="95"/>
+</segment>
+</net>
+<net name="RPI_SIGNAL_2" class="0">
+<segment>
+<pinref part="X1" gate="G$1" pin="GPIO26"/>
+<wire x1="91.44" y1="20.32" x2="86.36" y2="20.32" width="0.1524" layer="91"/>
+<label x="68.58" y="20.32" size="1.778" layer="95"/>
+</segment>
+<segment>
 <pinref part="IC1" gate="PORTB_L" pin="PB3"/>
 <wire x1="22.86" y1="83.82" x2="27.94" y2="83.82" width="0.1524" layer="91"/>
 <label x="25.4" y="83.82" size="1.778" layer="95"/>
 </segment>
-<segment>
-<pinref part="X1" gate="G$1" pin="GPIO20"/>
-<wire x1="91.44" y1="17.78" x2="86.36" y2="17.78" width="0.1524" layer="91"/>
-<label x="68.58" y="17.78" size="1.778" layer="95"/>
-</segment>
-</net>
-<net name="RPI_SIGNAL_3" class="0">
-<segment>
-<pinref part="IC1" gate="PORTB_L" pin="PB4"/>
-<wire x1="22.86" y1="81.28" x2="27.94" y2="81.28" width="0.1524" layer="91"/>
-<label x="25.4" y="81.28" size="1.778" layer="95"/>
-</segment>
-<segment>
-<pinref part="X1" gate="G$1" pin="GPIO16"/>
-<wire x1="91.44" y1="22.86" x2="86.36" y2="22.86" width="0.1524" layer="91"/>
-<label x="68.58" y="22.86" size="1.778" layer="95"/>
-</segment>
-</net>
-<net name="RPI_SIGNAL_2" class="0">
+</net>
+<net name="RPI_SIGNAL_1" class="0">
+<segment>
+<pinref part="X1" gate="G$1" pin="GPIO19"/>
+<wire x1="91.44" y1="25.4" x2="86.36" y2="25.4" width="0.1524" layer="91"/>
+<label x="68.58" y="25.4" size="1.778" layer="95"/>
+</segment>
 <segment>
 <pinref part="IC1" gate="PORTB_L" pin="PB5"/>
@@
 <label x="25.4" y="78.74" size="1.778" layer="95"/>
 </segment>
-<segment>
-<pinref part="X1" gate="G$1" pin="GPIO26"/>
-<wire x1="91.44" y1="20.32" x2="86.36" y2="20.32" width="0.1524" layer="91"/>
-<label x="68.58" y="20.32" size="1.778" layer="95"/>
-</segment>
-</net>
-<net name="RPI_SIGNAL_1" class="0">
-<segment>
-<pinref part="IC1" gate="PORTB_L" pin="PB6"/>
-<wire x1="22.86" y1="76.2" x2="27.94" y2="76.2" width="0.1524" layer="91"/>
-<label x="25.4" y="76.2" size="1.778" layer="95"/>
-</segment>
-<segment>
-<pinref part="X1" gate="G$1" pin="GPIO19"/>
-<wire x1="91.44" y1="25.4" x2="86.36" y2="25.4" width="0.1524" layer="91"/>
-<label x="68.58" y="25.4" size="1.778" layer="95"/>
-</segment>
-</net>
+</net>
